File: ptt_board/ptt_board_debug/ptt_board_debug.kicad_pcb (KiCad board)
At the start: 2 copper layers, 59 x 39.2 mm, 13 parts, among them CN1 HX JN1.27-2X5P ZZ H4.9, J1 Conn_01x02_Pin, J2 Conn_01x02_Pin, P0.26 TestPoint, U1 SKB369

Commit message: [Housekeeping] Renamed project library
Parts:
- BT1: footprint Project_components:BAT-SMD_MY-1632-03 -> PTT_Project_library:BAT-SMD_MY-1632-03
- C1, C2: footprint Project_components:C0603 -> PTT_Project_library:C0603
- CN1: footprint Project_components:CONN-TH_10P-P1.27_HX-JN1.27-2X5P-ZZ-H4.9 -> PTT_Project_library:CONN-TH_10P-P1.27_HX-JN1.27-2X5P-ZZ-H4.9
- REF**: footprint Project_components:Push button C2927788 -> PTT_Project_library:Push button C2927788
- U1: footprint Project_components:SKYLAB_SKB369 -> PTT_Project_library:SKYLAB_SKB369
Changed lines of the file:
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@@
 		)
 	)
-	(footprint "Project_components:BAT-SMD_MY-1632-03"
+	(footprint "PTT_Project_library:BAT-SMD_MY-1632-03"
 		(layer "F.Cu")
 		(at 145 73 90)
@@
 		)
 		(embedded_fonts no)
-		(model "/home/robin/Projects/PTT/PTT_Kicad/PTT_PCB_v4/libraries/Project_components.3dshapes/BAT-SMD_MY-1632-03.wrl"
+		(model "/home/robin/Projects/PTT/PTT_Kicad/PTT_PCB_v4/libraries/PTT_Project_library.3dshapes/BAT-SMD_MY-1632-03.wrl"
 			(offset
 				(xyz 0 1.17 0)
@@
 		(embedded_fonts no)
 	)
-	(footprint "Project_components:C0603"
+	(footprint "PTT_Project_library:C0603"
 		(layer "F.Cu")
 		(at 99.2 70.49 180)
@@
 		)
 		(embedded_fonts no)
-		(model "/home/robin/Projects/PTT/PTT_Kicad/PTT_PCB_v4/libraries/Project_components.3dshapes/C0603_L1.6-W0.8-H0.8.wrl"
+		(model "/home/robin/Projects/PTT/PTT_Kicad/PTT_PCB_v4/libraries/PTT_Project_library.3dshapes/C0603_L1.6-W0.8-H0.8.wrl"
 			(offset
 				(xyz -0.5 -0.13 -0)
@@
 		(embedded_fonts no)
 	)
-	(footprint "Project_components:Push button C2927788"
+	(footprint "PTT_Project_library:Push button C2927788"
 		(layer "F.Cu")
 		(at 99.4 78.2 90)
@@
 		)
 		(embedded_fonts no)
-		(model "/home/robin/Projects/PTT/PTT_Kicad/PTT_PCB_v4/libraries/Project_components.3dshapes/SW-SMD_4P-L5.1-W5.1-P3.70-LS6.5-TL_H1.5.wrl"
+		(model "/home/robin/Projects/PTT/PTT_Kicad/PTT_PCB_v4/libraries/PTT_Project_library.3dshapes/SW-SMD_4P-L5.1-W5.1-P3.70-LS6.5-TL_H1.5.wrl"
 			(offset
 				(xyz 0 -0 -0)
@@
 		)
 	)
-	(footprint "Project_components:SKYLAB_SKB369"
+	(footprint "PTT_Project_library:SKYLAB_SKB369"
 		(layer "F.Cu")
 		(at 118.45 73.48)
@@
 		(embedded_fonts no)
 	)
-	(footprint "Project_components:C0603"
+	(footprint "PTT_Project_library:C0603"
 		(layer "F.Cu")
 		(at 99.2 73.49)
@@
 		)
 		(embedded_fonts no)
-		(model "/home/robin/Projects/PTT/PTT_Kicad/PTT_PCB_v4/libraries/Project_components.3dshapes/C0603_L1.6-W0.8-H0.8.wrl"
+		(model "/home/robin/Projects/PTT/PTT_Kicad/PTT_PCB_v4/libraries/PTT_Project_library.3dshapes/C0603_L1.6-W0.8-H0.8.wrl"
 			(offset
 				(xyz -0.5 -0.13 -0)
@@
 		)
 	)
-	(footprint "Project_components:CONN-TH_10P-P1.27_HX-JN1.27-2X5P-ZZ-H4.9"
+	(footprint "PTT_Project_library:CONN-TH_10P-P1.27_HX-JN1.27-2X5P-ZZ-H4.9"
 		(layer "F.Cu")
 		(at 117.29 94.39)
@@
 		)
 		(embedded_fonts no)
-		(model "/home/robin/Projects/PTT/PTT_Kicad/PTT_PCB_v4/libraries/Project_components.3dshapes/CONN-TH_10P-P1.27_DC3-10P.wrl"
+		(model "/home/robin/Projects/PTT/PTT_Kicad/PTT_PCB_v4/libraries/PTT_Project_library.3dshapes/CONN-TH_10P-P1.27_DC3-10P.wrl"
 			(offset
 				(xyz 0 -0 0)
