File: radio_board/radio_board.kicad_sch (KiCad schematic)
At the start: 88 parts, among them CN1 HX JN1.27-2X5P ZZ H4.9, Q1 2N7002K, SW2 RKB2SJG250SMTRLFS, SW3 MSK12C02, U1 FSC-BT1036C, U2 TP4057, U3 XB5352A, U5 S2B-PH-K-S(LF)(SN), U6 TLV75533PDBVR, U7 LMV321, U8 STM32G030F6P6TR

Commit message: [WIP]
Parts:
- removed C31: 100nF, Resistor_SMD:R_0603_1608Metric_Pad0.98x0.95mm_HandSolder, symbol Device:C
- removed R20: 10K, Resistor_SMD:R_0603_1608Metric_Pad0.98x0.95mm_HandSolder, symbol Device:R
- added R21: 150K, Resistor_SMD:R_0603_1608Metric_Pad0.98x0.95mm_HandSolder, symbol Device:R
- added R22: 100K, Resistor_SMD:R_0603_1608Metric_Pad0.98x0.95mm_HandSolder, symbol Device:R
- added R23: Poka Yoke UART, poka_yuke:poka_yoke_uart_Solder, symbol poka_yoke:Poka Yoke UART
Connections:
- net +BATT: now also R22.1; no longer U8.12 (PA5)
- net GND: now also R16.1, R21.1; no longer R16.2
- net UART_RX: now also R23.3; no longer U8.20 (PB3/PB4/PB5/PB6)
- net UART_TX: now also R23.1; no longer U8.1 (PB7/PB8)
- net at C20.2, RV1.3: now also R16.2; no longer R16.1
- net RESET_FSC: no longer names the net of U8.9 (PA2)
- net RESET_FSC: no longer U1.8 (RESET)
- new net: R23.4, U8.1 (PB7/PB8)
- new net: R21.2, R22.2, U8.12 (PA5)
- new net: R23.2, U8.20 (PB3/PB4/PB5/PB6)
Other:
- moved on the sheet: C30, C8, C9, D5, R18, R19, SW2, U8

Commit message: [WIP]
Parts:
- removed CN1: HX JN1.27-2X5P ZZ H4.9, PTT_Project_library:CONN-TH_10P-P1.27_HX-JN1.27-2X5P-ZZ-H4.9, symbol PTT_Project_library:HXJN1.27-2X5PZZH4.9
- removed TP52: Debug_gpio, TestPoint:TestPoint_THTPad_D2.0mm_Drill1.0mm, symbol Connector:TestPoint
- added J1: 3.3v, Connector_PinSocket_2.54mm:PinSocket_1x01_P2.54mm_Vertical, symbol Connector:Conn_01x01_Pin
- added J2: GND, Connector_PinSocket_2.54mm:PinSocket_1x01_P2.54mm_Vertical, symbol Connector:Conn_01x01_Pin
- added J3: RESET, Connector_PinSocket_2.54mm:PinSocket_1x01_P2.54mm_Vertical, symbol Connector:Conn_01x01_Pin
- added J4: SWDCLK, Connector_PinSocket_2.54mm:PinSocket_1x01_P2.54mm_Vertical, symbol Connector:Conn_01x01_Pin
- added J5: SWDIO, Connector_PinSocket_2.54mm:PinSocket_1x01_P2.54mm_Vertical, symbol Connector:Conn_01x01_Pin
- added R20: 1, Resistor_SMD:R_0603_1608Metric_Pad0.98x0.95mm_HandSolder, symbol Device:R
- added TP1: TP_IBATT_H, TestPoint:TestPoint_THTPad_D2.0mm_Drill1.0mm, symbol Connector:TestPoint
- added TP3: TP_IBATT_L, TestPoint:TestPoint_THTPad_D2.0mm_Drill1.0mm, symbol Connector:TestPoint
- TP47: footprint TestPoint:TestPoint_Pad_D3.0mm -> TestPoint:TestPoint_Pad_D2.5mm
- TP6: footprint TestPoint:TestPoint_THTPad_D2.0mm_Drill1.0mm -> TestPoint:TestPoint_Pad_D2.5mm
Connections:
- net +3.3V: now also J1.1 (Pin_1); no longer SW2.2
- net +BATT: now also R20.2, TP3.1; no longer TP47.1, U5.2
- net GND: now also SW2.2, J2.1 (Pin_1)
- net RESET: now also J3.1 (Pin_1)
- net SWDCLK: now also J4.1 (Pin_1)
- net SWDIO: now also J5.1 (Pin_1)
- net UART_TX: now also R23.4; no longer R23.1
- net at U8.1 (PB7/PB8): now also R23.1; no longer R23.4
- net at U8.11 (PA4): now also SW2.3; no longer SW2.4
- net MIC_BIAS: no longer names the net of U1.45 (MIC_BIAS)
- new net: R20.1, TP1.1, TP47.1, U5.2
Other:
- moved on the sheet: SW2, U5
