File: ptt_board/ptt_board_cell/ptt_board_cell.kicad_pcb (KiCad board)
At the start: 2 copper layers, 26.4 x 26.4 mm, 4 parts, among them P26 Conn_01x01_Pin

Commit message: [WIP]
Parts:
- removed P26: Conn_01x01_Pin, Connector_Pin:Pin_D1.0mm_L10.0mm
- added Batt2: Conn_01x01_Pin, Connector_Pin:Pin_D1.0mm_L10.0mm, F.Cu at (142.5, 109.5)
- added Gnd1: Conn_01x01_Pin, Connector_Pin:Pin_D1.0mm_L10.0mm, F.Cu at (147.5, 100.8)
- added P019: Conn_01x01_Pin, Connector_Pin:Pin_D1.0mm_L10.0mm, F.Cu at (124.8, 100.8)
- added P19: Conn_01x01_Pin, Connector_Pin:Pin_D1.0mm_L10.0mm, F.Cu at (88.8, 100.8)
- moved BAT1 37.3 mm to (136.0, 100.5), turned to 0 degrees
Connections:
- BAT1 pad 1: (no net) -> +BATT
- BAT1 pad 2: (no net) -> GND
Other:
- board size 26.4 x 26.4 mm -> 62.4 x 27.8 mm

Commit message: [WIP]
Parts:
- removed BAT1: MY-2032-22, Project_components:BAT-TH_MY-2032-22
- removed the Batt2 at (142.5, 109.5)
- removed the Batt2 at (106.5, 109.5)
- removed the Gnd1 at (111.5, 100.8)
- removed the Gnd1 at (147.5, 100.8)
- removed P019: Conn_01x01_Pin, Connector_Pin:Pin_D1.0mm_L10.0mm
- added Batt2: Conn_01x01_Pin, Connector_PinHeader_2.54mm:PinHeader_1x01_P2.54mm_Vertical, F.Cu at (106.8, 109.4)
- added Gnd1: Conn_01x01_Pin, Connector_PinHeader_2.54mm:PinHeader_1x01_P2.54mm_Vertical, F.Cu at (110.0, 93.6)
- added U1: MY-2032-02, Project_components:BATT-TH_MY-2032-02, B.Cu at (100.0, 100.0)
- P19: footprint Connector_Pin:Pin_D1.0mm_L10.0mm -> Connector_PinHeader_2.54mm:PinHeader_1x01_P2.54mm_Vertical
- moved P19 3.26 mm to (89.0, 104.0)
Other:
- board size 62.4 x 27.8 mm -> 26.4 x 26.4 mm

Commit message: [WIP]
Parts:
- moved Gnd1 20.8 mm to (89.2, 95.2)
- moved Batt2 0.46 mm to (106.5, 109.8)
- moved P19 0.25 mm to (89.2, 104.0)
- turned U1 to -38 degrees
Routing:
- net GND: track 0.00 -> 14.0 mm
Other:
- board size 26.4 x 26.4 mm -> 26.8 x 26.4 mm
- board text added: "Gnd1"

Commit message: [Housekeeping] Renamed project library
Parts:
- U1: footprint Project_components:BATT-TH_MY-2032-02 -> PTT_Project_library:BATT-TH_MY-2032-02
Changed lines of the file:
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@@
 		)
 	)
-	(footprint "Project_components:BATT-TH_MY-2032-02"
+	(footprint "PTT_Project_library:BATT-TH_MY-2032-02"
 		(layer "B.Cu")
 		(at 100 100 -38)
@@
 		)
 		(embedded_fonts no)
-		(model "/home/rbaruffa/Perso/OmniPTT/hardware/libraries/Project_components.3dshapes/BATT-TH_MY-2032-02.wrl"
+		(model "/home/rbaruffa/Perso/OmniPTT/hardware/libraries/PTT_Project_library.3dshapes/BATT-TH_MY-2032-02.wrl"
 			(offset
 				(xyz 0 0 0)

Commit message: [Milestone] Last commit before pourchasing v2
Routing:
- net GND: track 14.0 -> 12.7 mm
Other:
- board size 26.8 x 26.4 mm -> 26.1 x 26.4 mm
- board text removed: "Gnd1"
Changed lines of the file:
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@@
 			(outputformat 1)
 			(mirror no)
-			(drillshape 1)
+			(drillshape 0)
 			(scaleselection 1)
-			(outputdirectory "")
+			(outputdirectory "exports/gerber/")
 		)
 	)
@@
 		(tags "Through hole pin header THT 1x01 2.54mm single row")
 		(property "Reference" "P19"
-			(at 3.8 0.2 0)
+			(at 3.75 0.5 0)
 			(layer "F.SilkS")
 			(effects
@@
 			)
 		)
+		(property ki_fp_filters "Connector*:*_1x??_*")
+		(sheetname "/")
+		(sheetfile "ptt_board_cell.kicad_sch")
 		(attr through_hole)
 		(fp_line
@@
 			(layer "F.Fab")
 		)
-		(fp_text user "${REFERENCE}"
-			(at 0 0 90)
-			(layer "F.Fab")
-			(effects
-				(font
-					(size 1 1)
-					(thickness 0.15)
-				)
-			)
-		)
 		(pad "1" thru_hole circle
 			(at 0 0)
 			(size 1.7 1.7)
-			(drill 1)
+			(drill 0.95)
 			(layers "*.Cu" "*.Mask")
 			(remove_unused_layers no)
@@
 		(tags "Through hole pin header THT 1x01 2.54mm single row")
 		(property "Reference" "Gnd1"
-			(at -4.2 0.4 0)
+			(at 3.75 0.5 0)
 			(layer "F.SilkS")
 			(effects
@@
 			)
 		)
+		(property ki_fp_filters "Connector*:*_1x??_*")
+		(sheetname "/")
+		(sheetfile "ptt_board_cell.kicad_sch")
 		(attr through_hole)
 		(fp_line
@@
 			(layer "F.Fab")
 		)
-		(fp_text user "${REFERENCE}"
-			(at 0 0 90)
-			(layer "F.Fab")
-			(effects
-				(font
-					(size 1 1)
-					(thickness 0.15)
-				)
-			)
-		)
 		(pad "1" thru_hole circle
 			(at 0 0)
 			(size 1.7 1.7)
-			(drill 1)
+			(drill 0.95)
 			(layers "*.Cu" "*.Mask")
 			(remove_unused_layers no)
@@
 		(tags "Through hole pin header THT 1x01 2.54mm single row")
 		(property "Reference" "Batt2"
-			(at -0.2 -3.4 0)
+			(at -4.5 0.25 0)
 			(layer "F.SilkS")
 			(effects
@@
 			)
 		)
+		(property ki_fp_filters "Connector*:*_1x??_*")
+		(sheetname "/")
+		(sheetfile "ptt_board_cell.kicad_sch")
 		(attr through_hole)
 		(fp_line
@@
 			(layer "F.Fab")
 		)
-		(fp_text user "${REFERENCE}"
-			(at 0 0 90)
-			(layer "F.Fab")
-			(effects
-				(font
-					(size 1 1)
-					(thickness 0.15)
-				)
-			)
-		)
 		(pad "1" thru_hole circle
 			(at 0 0)
 			(size 1.7 1.7)
-			(drill 1)
+			(drill 0.95)
 			(layers "*.Cu" "*.Mask")
 			(remove_unused_layers no)
@@
 		(net 1)
 	)
-	(gr_rect
-		(start 86.6 98)
-		(end 89.6 102)
-		(stroke
-			(width 0.2)
-			(type solid)
-		)
-		(fill no)
-		(layer "Edge.Cuts")
-	)
-	(gr_circle
-		(center 100 100)
-		(end 113.2 100)
-		(stroke
-			(width 0.2)
-			(type solid)
+	(gr_poly
+		(pts
+			(xy 100.40651 86.80576) (xy 100.731459 86.81978) (xy 101.055964 86.841802) (xy 101.379828 86.871813)
+			(xy 101.702854 86.909793) (xy 102.024847 86.955721) (xy 102.34561 87.009567) (xy 102.664949 87.0713)
+			(xy 102.98267 87.140882) (xy 103.298581 87.218271) (xy 103.612489 87.30342) (xy 103.924203 87.396276)
+			(xy 104.233536 87.496784) (xy 104.540298 87.604883) (xy 104.844304 87.720507) (xy 105.145369 87.843586)
+			(xy 105.44331 87.974045) (xy 105.737947 88.111804) (xy 106.0291 88.256781) (xy 106.316592 88.408888)
+			(xy 106.600251 88.568031) (xy 106.879902 88.734114) (xy 107.155376 88.907037) (xy 107.426506 89.086695)
+			(xy 107.693128 89.272978) (xy 107.955079 89.465773) (xy 108.212201 89.664963) (xy 108.464337 89.870428)
+			(xy 108.711334 90.082043) (xy 108.953043 90.299678) (xy 109.189317 90.523203) (xy 109.420012 90.752481)
+			(xy 109.644987 90.987373) (xy 109.864108 91.227737) (xy 110.07724 91.473426) (xy 110.284254 91.724292)
+			(xy 110.485024 91.980182) (xy 110.67943 92.24094) (xy 110.867351 92.506409) (xy 111.048676 92.776428)
+			(xy 111.223292 93.050832) (xy 111.391095 93.329454) (xy 111.551983 93.612127) (xy 111.705857 93.898677)
+			(xy 111.852625 94.188932) (xy 111.992197 94.482714) (xy 112.124488 94.779846) (xy 112.249419 95.080147)
+			(xy 112.366914 95.383435) (xy 112.4769 95.689525) (xy 112.579312 95.998233) (xy 112.674087 96.30937)
+			(xy 112.761167 96.622747) (xy 112.840501 96.938175) (xy 112.912038 97.255462) (xy 112.975737 97.574414)
+			(xy 113.031559 97.89484) (xy 113.04722 98) (xy 110.4 98) (xy 110.4 102) (xy 113.04722 102) (xy 113.031559 102.10516)
+			(xy 112.975737 102.425586) (xy 112.912038 102.744538) (xy 112.840501 103.061825) (xy 112.761167 103.377253)
+			(xy 112.674087 103.69063) (xy 112.579312 104.001767) (xy 112.4769 104.310475) (xy 112.366914 104.616565)
+			(xy 112.249419 104.919853) (xy 112.124488 105.220154) (xy 111.992197 105.517286) (xy 111.852625 105.811068)
+			(xy 111.705857 106.101323) (xy 111.551983 106.387873) (xy 111.391095 106.670546) (xy 111.223292 106.949168)
+			(xy 111.048676 107.223572) (xy 110.867351 107.493591) (xy 110.67943 107.75906) (xy 110.485024 108.019818)
+			(xy 110.284254 108.275708) (xy 110.07724 108.526574) (xy 109.864108 108.772263) (xy 109.644987 109.012627)
+			(xy 109.420012 109.247519) (xy 109.189317 109.476797) (xy 108.953043 109.700322) (xy 108.711334 109.917957)
+			(xy 108.464337 110.129572) (xy 108.212201 110.335037) (xy 107.955079 110.534227) (xy 107.693128 110.727022)
+			(xy 107.426506 110.913305) (xy 107.155376 111.092963) (xy 106.879902 111.265886) (xy 106.600251 111.431969)
+			(xy 106.316592 111.591112) (xy 106.0291 111.743219) (xy 105.737947 111.888196) (xy 105.44331 112.025955)
+			(xy 105.145369 112.156414) (xy 104.844304 112.279493) (xy 104.540298 112.395117) (xy 104.233536 112.503216)
+			(xy 103.924203 112.603724) (xy 103.612489 112.69658) (xy 103.298581 112.781729) (xy 102.98267 112.859118)
+			(xy 102.664949 112.9287) (xy 102.34561 112.990433) (xy 102.024847 113.044279) (xy 101.702854 113.090207)
+			(xy 101.379828 113.128187) (xy 101.055964 113.158198) (xy 100.731459 113.18022) (xy 100.40651 113.19424)
+			(xy 100.081314 113.200251) (xy 99.756069 113.198247) (xy 99.430972 113.188231) (xy 99.10622 113.170208)
+			(xy 98.782011 113.14419) (xy 98.458542 113.110192) (xy 98.136008 113.068235) (xy 97.814606 113.018344)
+			(xy 97.49453 112.96055) (xy 97.175976 112.894887) (xy 96.859136 112.821396) (xy 96.544203 112.740121)
+			(xy 96.231368 112.651112) (xy 95.920821 112.554422) (xy 95.61275 112.450111) (xy 95.307343 112.338241)
+			(xy 95.004785 112.218881) (xy 94.705259 112.092102) (xy 94.408947 111.957983) (xy 94.11603 111.816604)
+			(xy 93.826685 111.668051) (xy 93.541088 111.512414) (xy 93.259412 111.349789) (xy 92.981829 111.180273)
+			(xy 92.708506 111.003969) (xy 92.439609 110.820985) (xy 92.175303 110.631432) (xy 91.915746 110.435424)
+			(xy 91.661098 110.233081) (xy 91.411512 110.024525) (xy 91.167141 109.809884) (xy 90.928131 109.589287)
+			(xy 90.69463 109.362869) (xy 90.466777 109.130766) (xy 90.244712 108.89312) (xy 90.028569 108.650075)
+			(xy 89.81848 108.401779) (xy 89.614573 108.148382) (xy 89.41697 107.890038) (xy 89.225792 107.626904)
+			(xy 89.041155 107.35914) (xy 88.863171 107.086908) (xy 88.691948 106.810374) (xy 88.52759 106.529705)
+			(xy 88.370198 106.245072) (xy 88.219865 105.956648) (xy 88.076684 105.664607) (xy 87.940742 105.369127)
+			(xy 87.812121 105.070388) (xy 87.690899 104.768571) (xy 87.57715 104.463859) (xy 87.470943 104.156436)
+			(xy 87.372342 103.846491) (xy 87.281408 103.53421) (xy 87.198195 103.219783) (xy 87.122753 102.903402)
+			(xy 87.05513 102.585258) (xy 86.995365 102.265545) (xy 86.952468 102) (xy 89.6 102) (xy 89.6 98)
+			(xy 86.952468 98) (xy 86.995365 97.734455) (xy 87.05513 97.414742) (xy 87.122753 97.096598) (xy 87.198195 96.780217)
+			(xy 87.281408 96.46579) (xy 87.372342 96.153509) (xy 87.470943 95.843564) (xy 87.57715 95.536141)
+			(xy 87.690899 95.231429) (xy 87.812121 94.929612) (xy 87.940742 94.630873) (xy 88.076684 94.335393)
+			(xy 88.219865 94.043352) (xy 88.370198 93.754928) (xy 88.52759 93.470295) (xy 88.691948 93.189626)
+			(xy 88.863171 92.913092) (xy 89.041155 92.64086) (xy 89.225792 92.373096) (xy 89.41697 92.109962)
+			(xy 89.614573 91.851618) (xy 89.81848 91.598221) (xy 90.028569 91.349925) (xy 90.244712 91.10688)
+			(xy 90.466777 90.869234) (xy 90.69463 90.637131) (xy 90.928131 90.410713) (xy 91.167141 90.190116)
+			(xy 91.411512 89.975475) (xy 91.661098 89.766919) (xy 91.915746 89.564576) (xy 92.175303 89.368568)
+			(xy 92.439609 89.179015) (xy 92.708506 88.996031) (xy 92.981829 88.819727) (xy 93.259412 88.650211)
+			(xy 93.541088 88.487586) (xy 93.826685 88.331949) (xy 94.11603 88.183396) (xy 94.408947 88.042017)
+			(xy 94.705259 87.907898) (xy 95.004785 87.781119) (xy 95.307343 87.661759) (xy 95.61275 87.549889)
+			(xy 95.920821 87.445578) (xy 96.231368 87.348888) (xy 96.544203 87.259879) (xy 96.859136 87.178604)
+			(xy 97.175976 87.105113) (xy 97.49453 87.03945) (xy 97.814606 86.981656) (xy 98.136008 86.931765)
+			(xy 98.458542 86.889808) (xy 98.782011 86.85581) (xy 99.10622 86.829792) (xy 99.430972 86.811769)
+			(xy 99.756069 86.801753) (xy 100.081314 86.799749)
 		)
-		(fill no)
-		(layer "Edge.Cuts")
-	)
-	(gr_rect
-		(start 110.4 98)
-		(end 113.4 102)
 		(stroke
 			(width 0.2)
-			(type solid)
+			(type default)
 		)
 		(fill no)
 		(layer "Edge.Cuts")
 	)
-	(gr_text "Gnd1"
-		(at 89.25 95.25 90)
-		(layer "F.Fab")
-		(effects
-			(font
-				(size 1 1)
-				(thickness 0.15)
-			)
-		)
-	)
-	(segment
-		(start 109.85 94.05)
-		(end 110 93.9)
-		(width 1)
-		(layer "B.Cu")
-		(net 2)
-	)
-	(segment
-		(start 110 93.9)
-		(end 109.85 93.75)
-		(width 0.2)
-		(layer "B.Cu")
-		(net 2)
-	)
 	(segment
 		(start 100 100)
-		(end 106 100)
-		(width 1)
-		(layer "B.Cu")
-		(net 2)
-	)
-	(segment
-		(start 106 100)
-		(end 109.85 96.15)
+		(end 94 100)
 		(width 1)
 		(layer "B.Cu")
@@
 	)
 	(segment
-		(start 109.85 96.15)
-		(end 109.85 94.05)
+		(start 94 100)
+		(end 89.25 95.25)
 		(width 1)
 		(layer "B.Cu")
