File: ptt_board/ptt_board_cell/ptt_board_cell.kicad_sch (KiCad schematic)
At the start: 5 parts, among them SW1 RKB2SJG250SMTRLFS

Commit message: [WIP] Started net rev of ptt board and radio board
Parts:
- removed CLK1: Conn_01x01_Pin, Connector_PinHeader_2.54mm:PinHeader_1x01_P2.54mm_Vertical, symbol Connector:Conn_01x01_Pin
- removed SW1: RKB2SJG250SMTRLFS, PTT_project:Push button C2927788, symbol Project_components:RKB2SJG250SMTRLFS
- added BAT1: MY-2032-22, Project_components:BAT-TH_MY-2032-22, symbol PTT_project:MY-2032-22
- Batt2: renamed from IO1; footprint Connector_PinHeader_2.54mm:PinHeader_1x01_P2.54mm_Vertical -> Connector_Pin:Pin_D1.0mm_L10.0mm
- Gnd1: footprint Connector_PinHeader_2.54mm:PinHeader_1x01_P2.54mm_Vertical -> Connector_Pin:Pin_D1.0mm_L10.0mm
- P26: renamed from Bat1; footprint Connector_PinHeader_2.54mm:PinHeader_1x01_P2.54mm_Vertical -> Connector_Pin:Pin_D1.0mm_L10.0mm
Connections:
- net GND: now reaches Gnd1.1 (Pin_1)
- net GND: now also BAT1.2
- net SWDIO renamed +BATT
- net +BATT: now also BAT1.1

Commit message: [WIP]
Parts:
- renumbered P26 to P19
Changed lines of the file:
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@@
 		(on_board yes)
 		(dnp no)
-		(property "Reference" "P26"
+		(property "Reference" "P19"
 			(at 189.865 55.88 0)
 			(effects
@@
 			(project "ptt_board_cell"
 				(path "/7b4c058f-fd9c-4c59-ad3d-5046394d5b15"
-					(reference "P26")
+					(reference "P19")
 					(unit 1)
 				)

Commit message: [WIP]
Parts:
- removed BAT1: MY-2032-22, Project_components:BAT-TH_MY-2032-22, symbol PTT_project:MY-2032-22
- added U1: MY-2032-02, Project_components:BATT-TH_MY-2032-02, symbol Project_components:MY-2032-02
- Batt2, Gnd1, P19: footprint Connector_Pin:Pin_D1.0mm_L10.0mm -> Connector_PinHeader_2.54mm:PinHeader_1x01_P2.54mm_Vertical
Connections:
- net +BATT: now also U1.1
- net GND: now also U1.2
Changed lines of the file:
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@@
 	(wire
 		(pts
-			(xy 199.39 63.5) (xy 205.74 63.5)
+			(xy 200.66 66.04) (xy 204.47 66.04)
 		)
 		(stroke
@@
 	(wire
 		(pts
-			(xy 181.61 63.5) (xy 189.23 63.5)
+			(xy 182.88 66.04) (xy 187.96 66.04)
 		)
 		(stroke
@@
 	(symbol
 		(lib_id "power:+BATT")
-		(at 181.61 63.5 90)
+		(at 182.88 66.04 90)
 		(unit 1)
 		(exclude_from_sim no)
@@
 		(fields_autoplaced yes)
 		(property "Reference" "#PWR05"
-			(at 185.42 63.5 0)
+			(at 186.69 66.04 0)
 			(effects
 				(font
@@
 		)
 		(property "Value" "+BATT"
-			(at 177.8 63.4999 90)
+			(at 179.07 66.0399 90)
 			(effects
 				(font
@@
 		)
 		(property "Footprint" ""
-			(at 181.61 63.5 0)
+			(at 182.88 66.04 0)
 			(effects
 				(font
@@
 		)
 		(property "Datasheet" ""
-			(at 181.61 63.5 0)
+			(at 182.88 66.04 0)
 			(effects
 				(font
@@
 		)
 		(property "Description" "Power symbol creates a global label with name \"+BATT\""
-			(at 181.61 63.5 0)
+			(at 182.88 66.04 0)
 			(effects
 				(font
@@
 	(symbol
 		(lib_id "power:GND")
-		(at 205.74 63.5 90)
+		(at 204.47 66.04 90)
 		(unit 1)
 		(exclude_from_sim no)
@@
 		(fields_autoplaced yes)
 		(property "Reference" "#PWR010"
-			(at 212.09 63.5 0)
+			(at 210.82 66.04 0)
 			(effects
 				(font
@@
 		)
 		(property "Value" "GND"
-			(at 209.55 63.4999 90)
+			(at 208.28 66.0399 90)
 			(effects
 				(font
@@
 		)
 		(property "Footprint" ""
-			(at 205.74 63.5 0)
+			(at 204.47 66.04 0)
 			(effects
 				(font
@@
 		)
 		(property "Datasheet" ""
-			(at 205.74 63.5 0)
+			(at 204.47 66.04 0)
 			(effects
 				(font
@@
 		)
 		(property "Description" "Power symbol creates a global label with name \"GND\" , ground"
-			(at 205.74 63.5 0)
+			(at 204.47 66.04 0)
 			(effects
 				(font
@@
 			)
 		)
-		(property "Footprint" "Connector_Pin:Pin_D1.0mm_L10.0mm"
+		(property "Footprint" "Connector_PinHeader_2.54mm:PinHeader_1x01_P2.54mm_Vertical"
 			(at 189.23 50.8 0)
 			(effects
@@
 	)
 	(symbol
+		(lib_id "Project_components:MY-2032-02")
+		(at 194.31 66.04 0)
+		(unit 1)
+		(exclude_from_sim no)
+		(in_bom yes)
+		(on_board yes)
+		(dnp no)
+		(fields_autoplaced yes)
+		(property "Reference" "U1"
+			(at 194.31 58.42 0)
+			(effects
+				(font
+					(size 1.27 1.27)
+				)
+			)
+		)
+		(property "Value" "MY-2032-02"
+			(at 194.31 60.96 0)
+			(effects
+				(font
+					(size 1.27 1.27)
+				)
+			)
+		)
+		(property "Footprint" "Project_components:BATT-TH_MY-2032-02"
+			(at 194.31 73.66 0)
+			(effects
+				(font
+					(size 1.27 1.27)
+				)
+				(hide yes)
+			)
+		)
+		(property "Datasheet" "https://www.lcsc.com/datasheet/C964822.pdf"
+			(at 194.31 76.2 0)
+			(effects
+				(font
+					(size 1.27 1.27)
+				)
+				(hide yes)
+			)
+		)
+		(property "Description" ""
+			(at 194.31 66.04 0)
+			(effects
+				(font
+					(size 1.27 1.27)
+				)
+				(hide yes)
+			)
+		)
+		(property "Manufacturer" "MYOUNG(美阳)"
+			(at 194.31 78.74 0)
+			(effects
+				(font
+					(size 1.27 1.27)
+				)
+				(hide yes)
+			)
+		)
+		(property "MPN" "MY-2032-02"
+			(at 194.31 81.28 0)
+			(effects
+				(font
+					(size 1.27 1.27)
+				)
+				(hide yes)
+			)
+		)
+		(property "LCSC Part" "C964822"
+			(at 194.31 83.82 0)
+			(effects
+				(font
+					(size 1.27 1.27)
+				)
+				(hide yes)
+			)
+		)
+		(pin "2"
+		)
+		(pin "1"
+		)
+		(instances
+			(project "ptt_board_cell"
+				(path "/7b4c058f-fd9c-4c59-ad3d-5046394d5b15"
+					(reference "U1")
+					(unit 1)
+				)
+			)
+		)
+	)
+	(symbol
 		(lib_id "Connector:Conn_01x01_Pin")
 		(at 189.23 46.99 0)
@@
 			)
 		)
-		(property "Footprint" "Connector_Pin:Pin_D1.0mm_L10.0mm"
+		(property "Footprint" "Connector_PinHeader_2.54mm:PinHeader_1x01_P2.54mm_Vertical"
 			(at 189.23 46.99 0)
 			(effects
@@
 			)
 		)
-		(property "Footprint" "Connector_Pin:Pin_D1.0mm_L10.0mm"
+		(property "Footprint" "Connector_PinHeader_2.54mm:PinHeader_1x01_P2.54mm_Vertical"
 			(at 189.23 54.61 0)
 			(effects
@@
 					(unit 1)
 				)
-			)
-		)
-	)
-	(symbol
-		(lib_id "PTT_project:MY-2032-22")
-		(at 194.31 63.5 0)
-		(unit 1)
-		(exclude_from_sim no)
-		(in_bom yes)
-		(on_board yes)
-		(dnp no)
-		(property "Reference" "BAT1"
-			(at 194.31 69.85 0)
-			(effects
-				(font
-					(size 1.27 1.27)
-				)
-			)
-		)
-		(property "Value" "MY-2032-22"
-			(at 194.31 72.39 0)
-			(effects
-				(font
-					(size 1.27 1.27)
-				)
-			)
-		)
-		(property "Footprint" "Project_components:BAT-TH_MY-2032-22"
-			(at 194.31 71.12 0)
-			(effects
-				(font
-					(size 1.27 1.27)
-				)
-				(hide yes)
-			)
-		)
-		(property "Datasheet" "https://www.lcsc.com/datasheet/C2902339.pdf"
-			(at 194.31 73.66 0)
-			(effects
-				(font
-					(size 1.27 1.27)
-				)
-				(hide yes)
-			)
-		)
-		(property "Description" ""
-			(at 194.31 63.5 0)
-			(effects
-				(font
-					(size 1.27 1.27)
-				)
-				(hide yes)
-			)
-		)
-		(property "Manufacturer" "MYOUNG(美阳)"
-			(at 194.31 76.2 0)
-			(effects
-				(font
-					(size 1.27 1.27)
-				)
-				(hide yes)
-			)
-		)
-		(property "MPN" "MY-2032-22"
-			(at 194.31 78.74 0)
-			(effects
-				(font
-					(size 1.27 1.27)
-				)
-				(hide yes)
-			)
-		)
-		(property "LCSC Part" "C2902339"
-			(at 194.31 81.28 0)
-			(effects
-				(font
-					(size 1.27 1.27)
-				)
-				(hide yes)
-			)
-		)
-		(pin "1"
-		)
-		(pin "2"
-		)
-		(instances
-			(project "ptt_board_cell"
-				(path "/7b4c058f-fd9c-4c59-ad3d-5046394d5b15"
-					(reference "BAT1")
-					(unit 1)
-				)

Commit message: [Housekeeping] Renamed project library
Parts:
- U1: footprint Project_components:BATT-TH_MY-2032-02 -> PTT_Project_library:BATT-TH_MY-2032-02; symbol Project_components:MY-2032-02 -> PTT_Project_library:MY-2032-02
Changed lines of the file:
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@@
 	)
 	(symbol
-		(lib_id "Project_components:MY-2032-02")
+		(lib_id "PTT_Project_library:MY-2032-02")
 		(at 194.31 66.04 0)
 		(unit 1)
@@
 			)
 		)
-		(property "Footprint" "Project_components:BATT-TH_MY-2032-02"
+		(property "Footprint" "PTT_Project_library:BATT-TH_MY-2032-02"
 			(at 194.31 73.66 0)
 			(effects

Commit message: [Milestone] Last commit before pourchasing v2
Changed lines of the file:
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@@
+	)
+	(symbol
+		(lib_id "PTT_logo:LOGO")
+		(at 245.11 57.15 0)
+		(unit 1)
+		(exclude_from_sim no)
+		(in_bom yes)
+		(on_board yes)
+		(dnp no)
+		(fields_autoplaced yes)
+		(property "Reference" "#G1"
+			(at 245.11 14.4357 0)
+			(effects
+				(font
+					(size 1.27 1.27)
+				)
+				(hide yes)
+			)
+		)
+		(property "Value" "LOGO"
+			(at 245.11 99.8643 0)
+			(effects
+				(font
+					(size 1.27 1.27)
+				)
+				(hide yes)
+			)
+		)
+		(property "Footprint" "PTT_logo:omniPTT_logo"
+			(at 245.11 57.15 0)
+			(effects
+				(font
+					(size 1.27 1.27)
+				)
+				(hide yes)
+			)
+		)
+		(property "Datasheet" ""
+			(at 245.11 57.15 0)
+			(effects
+				(font
+					(size 1.27 1.27)
+				)
+				(hide yes)
+			)
+		)
+		(property "Description" ""
+			(at 245.11 57.15 0)
+			(effects
+				(font
+					(size 1.27 1.27)
+				)
+				(hide yes)
+			)
+		)
+		(instances
+			(project "ptt_board_cell"
+				(path "/7b4c058f-fd9c-4c59-ad3d-5046394d5b15"
+					(reference "#G1")
+					(unit 1)
+				)
+			)
+		)
 	)
 	(symbol
