File: ptt_board/ptt_board_core/ptt_board_core.kicad_sch (KiCad schematic)
At the start: 14 parts, among them P0.03 TestPoint, P0.07 TestPoint, P0.30 TestPoint, P26 Conn_01x01_Pin, U1 SKB369

Commit message: [WIP] Started net rev of ptt board and radio board
Parts:
- removed BT1: MY-1632-03-R, Project_components:BAT-SMD_MY-1632-03, symbol Project_components:MY-1632-03-R
- removed CLK1: Conn_01x01_Pin, Connector_PinHeader_2.54mm:PinHeader_1x01_P2.54mm_Vertical, symbol Connector:Conn_01x01_Pin
- removed P.0.31, P0.03, P0.07, P0.30, Reset1: TestPoint, TestPoint:TestPoint_Pad_D1.0mm, symbol Connector:TestPoint
- added CLK1, GND3, IO2, P0.26: TestPoint, TestPoint:TestPoint_Pad_D1.0mm, symbol Connector:TestPoint
- added R1: 470k, Resistor_SMD:R_0603_1608Metric_Pad0.98x0.95mm_HandSolder, symbol Device:R
- added SW1: RKB2SJG250SMTRLFS, Project_components:Push button C2927788, symbol Project_components:RKB2SJG250SMTRLFS
- Batt2: renamed from IO1; footprint Connector_PinHeader_2.54mm:PinHeader_1x01_P2.54mm_Vertical -> Connector_Pin:Pin_D1.0mm_L10.0mm
- Gnd1: footprint Connector_PinHeader_2.54mm:PinHeader_1x01_P2.54mm_Vertical -> Connector_Pin:Pin_D1.0mm_L10.0mm
- P026: renamed from P26; footprint Connector_PinHeader_2.54mm:PinHeader_1x01_P2.54mm_Vertical -> Connector_Pin:Pin_D1.0mm_L10.0mm
- renumbered Batt+1 to Batt1
Connections:
- net +BATT: now also Batt2.1 (Pin_1), SW1.4
- net GND: now also GND3.1, R1.2
- net SWDCLK: now also CLK1.1
- net SWDIO: now also IO2.1; no longer Batt2.1 (Pin_1)
- net P0.26: now reaches P026.1 (Pin_1), U1.4 (P0.26)
- net P0.26: now also P0.26.1, R1.1, SW1.2
- net P0.28: now reaches U1.6 (P0.28)
- net Reset: no longer names the net of U1.22 (P0.21/~{RESET})
Other:
- moved on the sheet: Batt1, C1, C2

Commit message: [WIP]
Parts:
- removed P0.26: TestPoint, TestPoint:TestPoint_Pad_D1.0mm, symbol Connector:TestPoint
- renumbered P026 to P019
Connections:
- net P0.19: now reaches U1.21 (P0.19)
- net P0.19: now also P019.1 (Pin_1), R1.1, SW1.2
- removed net P0.26: P019.1 (Pin_1), R1.1, SW1.2, U1.4 (P0.26)
- net P0.28: no longer names the net of U1.6 (P0.28)
Changed lines of the file:
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@@
-	(wire
-		(pts
-			(xy 124.46 88.9) (xy 129.54 88.9)
-		)
-		(stroke
-			(width 0)
-			(type default)
-		)
-	)
 	(wire
 		(pts
@@
 	(wire
 		(pts
-			(xy 167.64 50.8) (xy 172.72 50.8)
-		)
-		(stroke
-			(width 0)
-			(type default)
-		)
-	)
-	(wire
-		(pts
 			(xy 166.37 82.55) (xy 167.64 82.55)
 		)
@@
 	(wire
 		(pts
-			(xy 124.46 83.82) (xy 129.54 83.82)
+			(xy 83.82 93.98) (xy 88.9 93.98)
 		)
 		(stroke
@@
 		)
 	)
+	(global_label "P0.19"
+		(shape input)
+		(at 83.82 93.98 180)
+		(fields_autoplaced yes)
+		(effects
+			(font
+				(size 1.27 1.27)
+			)
+			(justify right)
+		)
+		(property "Intersheetrefs" "${INTERSHEET_REFS}"
+			(at 75.3315 93.98 0)
+			(effects
+				(font
+					(size 1.27 1.27)
+				)
+				(justify right)
+				(hide yes)
+			)
+		)
+	)
 	(global_label "SWDCLK"
 		(shape input)
@@
 		)
 	)
+	(global_label "P0.19"
+		(shape input)
+		(at 120.65 27.94 0)
+		(fields_autoplaced yes)
+		(effects
+			(font
+				(size 1.27 1.27)
+			)
+			(justify left)
+		)
+		(property "Intersheetrefs" "${INTERSHEET_REFS}"
+			(at 129.1385 27.94 0)
+			(effects
+				(font
+					(size 1.27 1.27)
+				)
+				(justify left)
+				(hide yes)
+			)
+		)
+	)
 	(global_label "SWDCLK"
 		(shape input)
@@
 		)
 	)
-	(global_label "P0.26"
+	(global_label "P0.19"
 		(shape input)
-		(at 129.54 88.9 0)
+		(at 172.72 24.13 0)
 		(fields_autoplaced yes)
 		(effects
@@
 		)
 		(property "Intersheetrefs" "${INTERSHEET_REFS}"
-			(at 138.0285 88.9 0)
-			(effects
-				(font
-					(size 1.27 1.27)
-				)
-				(justify left)
-				(hide yes)
-			)
-		)
-	)
-	(global_label "P0.26"
-		(shape input)
-		(at 120.65 27.94 0)
-		(fields_autoplaced yes)
-		(effects
-			(font
-				(size 1.27 1.27)
-			)
-			(justify left)
-		)
-		(property "Intersheetrefs" "${INTERSHEET_REFS}"
-			(at 129.1385 27.94 0)
-			(effects
-				(font
-					(size 1.27 1.27)
-				)
-				(justify left)
-				(hide yes)
-			)
-		)
-	)
-	(global_label "P0.26"
-		(shape input)
-		(at 172.72 50.8 0)
-		(fields_autoplaced yes)
-		(effects
-			(font
-				(size 1.27 1.27)
-			)
-			(justify left)
-		)
-		(property "Intersheetrefs" "${INTERSHEET_REFS}"
-			(at 181.2085 50.8 0)
-			(effects
-				(font
-					(size 1.27 1.27)
-				)
-				(justify left)
-				(hide yes)
-			)
-		)
-	)
-	(global_label "P0.26"
-		(shape input)
-		(at 172.72 24.13 0)
-		(fields_autoplaced yes)
-		(effects
-			(font
-				(size 1.27 1.27)
-			)
-			(justify left)
-		)
-		(property "Intersheetrefs" "${INTERSHEET_REFS}"
 			(at 181.2085 24.13 0)
-			(effects
-				(font
-					(size 1.27 1.27)
-				)
-				(justify left)
-				(hide yes)
-			)
-		)
-	)
-	(global_label "P0.28"
-		(shape input)
-		(at 129.54 83.82 0)
-		(fields_autoplaced yes)
-		(effects
-			(font
-				(size 1.27 1.27)
-			)
-			(justify left)
-		)
-		(property "Intersheetrefs" "${INTERSHEET_REFS}"
-			(at 138.0285 83.82 0)
 			(effects
 				(font
@@
 	(symbol
 		(lib_id "Connector:TestPoint")
-		(at 167.64 50.8 90)
-		(unit 1)
-		(exclude_from_sim no)
-		(in_bom yes)
-		(on_board yes)
-		(dnp no)
-		(property "Reference" "P0.26"
-			(at 159.004 50.8 90)
-			(effects
-				(font
-					(size 1.27 1.27)
-				)
-			)
-		)
-		(property "Value" "TestPoint"
-			(at 164.338 48.26 90)
-			(effects
-				(font
-					(size 1.27 1.27)
-				)
-				(hide yes)
-			)
-		)
-		(property "Footprint" "TestPoint:TestPoint_Pad_D1.0mm"
-			(at 167.64 45.72 0)
-			(effects
-				(font
-					(size 1.27 1.27)
-				)
-				(hide yes)
-			)
-		)
-		(property "Datasheet" "~"
-			(at 167.64 45.72 0)
-			(effects
-				(font
-					(size 1.27 1.27)
-				)
-				(hide yes)
-			)
-		)
-		(property "Description" "test point"
-			(at 167.64 50.8 0)
-			(effects
-				(font
-					(size 1.27 1.27)
-				)
-				(hide yes)
-			)
-		)
-		(pin "1"
-		)
-		(instances
-			(project "ptt_board_core"
-				(path "/9af4cf98-9d36-402b-9fdf-f0a46f53ba5a"
-					(reference "P0.26")
-					(unit 1)
-				)
-			)
-		)
-	)
-	(symbol
-		(lib_id "Connector:TestPoint")
 		(at 167.64 39.37 90)
 		(unit 1)
@@
 		(on_board yes)
 		(dnp no)
-		(property "Reference" "P026"
+		(property "Reference" "P019"
 			(at 164.465 29.21 0)
 			(effects
@@
 			(project "ptt_board_core"
 				(path "/9af4cf98-9d36-402b-9fdf-f0a46f53ba5a"
-					(reference "P026")
+					(reference "P019")
 					(unit 1)
 				)

Commit message: [WIP]
Parts:
- Batt2, Gnd1, P019: footprint Connector_Pin:Pin_D1.0mm_L10.0mm -> Connector_PinHeader_2.54mm:PinHeader_1x01_P2.54mm_Vertical
Changed lines of the file:
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@@
 			)
 		)
-		(property "Footprint" "Connector_Pin:Pin_D1.0mm_L10.0mm"
+		(property "Footprint" "Connector_PinHeader_2.54mm:PinHeader_1x01_P2.54mm_Vertical"
 			(at 163.83 24.13 0)
 			(effects
@@
 			)
 		)
-		(property "Footprint" "Connector_Pin:Pin_D1.0mm_L10.0mm"
+		(property "Footprint" "Connector_PinHeader_2.54mm:PinHeader_1x01_P2.54mm_Vertical"
 			(at 163.83 20.32 0)
 			(effects
@@
 			)
 		)
-		(property "Footprint" "Connector_Pin:Pin_D1.0mm_L10.0mm"
+		(property "Footprint" "Connector_PinHeader_2.54mm:PinHeader_1x01_P2.54mm_Vertical"
 			(at 163.83 27.94 0)
 			(effects

Commit message: [WIP]
Parts:
- C1, C2: footprint Project_components:C0603 -> Capacitor_SMD:C_0402_1005Metric_Pad0.74x0.62mm_HandSolder
Changed lines of the file:
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@@
 			)
 		)
-		(property "Footprint" "Project_components:C0603"
+		(property "Footprint" "Capacitor_SMD:C_0402_1005Metric_Pad0.74x0.62mm_HandSolder"
 			(at 172.72 77.47 0)
 			(effects
@@
 			)
 		)
-		(property "Footprint" "Project_components:C0603"
+		(property "Footprint" "Capacitor_SMD:C_0402_1005Metric_Pad0.74x0.62mm_HandSolder"
 			(at 172.72 74.93 0)
 			(effects

Commit message: [Housekeeping] Renamed project library
Parts:
- C1, C2: symbol Project_components:CC0603KRX7R9BB104 -> PTT_Project_library:CC0603KRX7R9BB104
- SW1: footprint Project_components:Push button C2927788 -> PTT_Project_library:Push button C2927788; symbol Project_components:RKB2SJG250SMTRLFS -> PTT_Project_library:RKB2SJG250SMTRLFS
- U1: footprint Project_components:SKYLAB_SKB369 -> PTT_Project_library:SKYLAB_SKB369; symbol Project_components:SKB369 -> PTT_Project_library:SKB369
Changed lines of the file:
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@@
 	)
 	(symbol
-		(lib_id "Project_components:CC0603KRX7R9BB104")
+		(lib_id "PTT_Project_library:CC0603KRX7R9BB104")
 		(at 172.72 69.85 0)
 		(unit 1)
@@
 	)
 	(symbol
-		(lib_id "Project_components:RKB2SJG250SMTRLFS")
+		(lib_id "PTT_Project_library:RKB2SJG250SMTRLFS")
 		(at 97.79 30.48 0)
 		(unit 1)
@@
 			)
 		)
-		(property "Footprint" "Project_components:Push button C2927788"
+		(property "Footprint" "PTT_Project_library:Push button C2927788"
 			(at 97.79 40.64 0)
 			(effects
@@
 	)
 	(symbol
-		(lib_id "Project_components:SKB369")
+		(lib_id "PTT_Project_library:SKB369")
 		(at 106.68 81.28 0)
 		(unit 1)
@@
 			)
 		)
-		(property "Footprint" "Project_components:SKYLAB_SKB369"
+		(property "Footprint" "PTT_Project_library:SKYLAB_SKB369"
 			(at 106.68 81.28 0)
 			(effects
@@
 	)
 	(symbol
-		(lib_id "Project_components:CC0603KRX7R9BB104")
+		(lib_id "PTT_Project_library:CC0603KRX7R9BB104")
 		(at 172.72 82.55 180)
 		(unit 1)

Commit message: [Feature] Cleaned up PCB and schematics. Add logo, checked schematic, layout and wiring
Parts:
- C1: value 0.1 uF -> 100nF
Changed lines of the file:
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@@
 			)
 		)
-		(property "Value" "0.1 uF"
+		(property "Value" "100nF"
 			(at 172.72 66.04 0)
 			(effects

Commit message: [Milestone] Last commit before pourchasing v2
Parts:
- Batt1, Batt2, CLK1, GND3, Gnd1, IO2, P019, SW1, U1: now left out of the parts list
- C1, C2: footprint Capacitor_SMD:C_0402_1005Metric_Pad0.74x0.62mm_HandSolder -> Capacitor_SMD:C_0603_1608Metric_Pad1.08x0.95mm_HandSolder
- R1: LCSC Part (none) -> C114622
Changed lines of the file:
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@@
+			)
+		)
+		(property "LCSC Part" "C114622"
+			(at 111.76 34.29 0)
+			(effects
+				(font
+					(size 1.27 1.27)
+				)
+				(hide yes)
 			)
 		)
@@
 			)
 		)
-		(property "Footprint" "Capacitor_SMD:C_0402_1005Metric_Pad0.74x0.62mm_HandSolder"
+		(property "Footprint" "Capacitor_SMD:C_0603_1608Metric_Pad1.08x0.95mm_HandSolder"
 			(at 172.72 77.47 0)
 			(effects
@@
 		(unit 1)
 		(exclude_from_sim no)
-		(in_bom yes)
+		(in_bom no)
 		(on_board yes)
 		(dnp no)
@@
 		(unit 1)
 		(exclude_from_sim no)
-		(in_bom yes)
+		(in_bom no)
 		(on_board yes)
 		(dnp no)
@@
 		(unit 1)
 		(exclude_from_sim no)
-		(in_bom yes)
+		(in_bom no)
 		(on_board yes)
 		(dnp no)
@@
 		(unit 1)
 		(exclude_from_sim no)
-		(in_bom yes)
+		(in_bom no)
 		(on_board yes)
 		(dnp no)
@@
 		(unit 1)
 		(exclude_from_sim no)
-		(in_bom yes)
+		(in_bom no)
 		(on_board yes)
 		(dnp no)
@@
 		(unit 1)
 		(exclude_from_sim no)
-		(in_bom yes)
+		(in_bom no)
 		(on_board yes)
 		(dnp no)
@@
 		(unit 1)
 		(exclude_from_sim no)
-		(in_bom yes)
+		(in_bom no)
 		(on_board yes)
 		(dnp no)
@@
 		(unit 1)
 		(exclude_from_sim no)
-		(in_bom yes)
+		(in_bom no)
 		(on_board yes)
 		(dnp no)
@@
 		(unit 1)
 		(exclude_from_sim no)
-		(in_bom yes)
+		(in_bom no)
 		(on_board yes)
 		(dnp no)
@@
 			)
 		)
-		(property "Footprint" "Capacitor_SMD:C_0402_1005Metric_Pad0.74x0.62mm_HandSolder"
+		(property "Footprint" "Capacitor_SMD:C_0603_1608Metric_Pad1.08x0.95mm_HandSolder"
 			(at 172.72 74.93 0)
 			(effects
